Commit message: merge example package into one

File: beckhoff_bringup/urdf/beckhoff_bot/beckhoff_bot_macro.ros2_control.xacro (robot description, xacro)
@@ -26,15 +26,14 @@
     <xacro:macro name="beckhoff_bot_ros2_control" params="
                 name
-                prefix
-                use_mock_hardware:=false
+                mock_hardware:=false
                 mock_sensor_commands:=false"
                 >
         <ros2_control name="${name}" type="system">
         <hardware>
-            <xacro:if value="${use_mock_hardware}">
+            <xacro:if value="${mock_hardware}">
                 <plugin>mock_components/GenericSystem</plugin>
                 <param name="mock_sensor_commands">${mock_sensor_commands}</param>
             </xacro:if>
-            <xacro:unless value="${use_mock_hardware}">
+            <xacro:unless value="${mock_hardware}">
                 <plugin>beckhoff_hardware_interface/BeckhoffSystem</plugin>
                 <param name="plc_ip_address">192.168.122.218</param>
@@ -49,4 +48,13 @@
         Declaring indices descending or out-of-order (2, 1, 0) causes mismatch between hw_states/command buffers and byte buffers received from PLC
         -->
+        <!-- These interfaces can be under any component - joint, gpio or sensor -->
+        <!-- Format
+            interface name - arbitrary
+            PLC_symbol - exact symbol in your Beckhoff PLC application
+            n_elements - elements in the PLC variable - defaults to 1
+            index - index of the element this interface is targeting in the PLC variable of type ARRAY[ ANY ]
+            PLC_type - type used to specify the byte size of the PLC variable
+            initial_value (command) - initial value written to the command
+            -->
         <gpio name="robot_io">
             <xacro:command_interface_PLC name="ManualJogging" PLC_symbol="MAIN.bManualJogging" PLC_type="BOOL" initial_value="1"/>

File: beckhoff_bringup/urdf/beckhoff_bot/beckhoff_bot_macro.xacro (robot description, xacro)
@@ -1,6 +1,6 @@
 <?xml version="1.0" encoding="UTF-8"?>
 <robot xmlns:xacro="http://wiki.ros.org/xacro">
-  <xacro:include filename="$(find beckhoff_description)/urdf/common/inertials.xacro"/>
-  <xacro:include filename="$(find beckhoff_description)/urdf/common/materials.xacro"/>
+  <xacro:include filename="$(find beckhoff_bringup)/urdf/common/inertials.xacro"/>
+  <xacro:include filename="$(find beckhoff_bringup)/urdf/common/materials.xacro"/>
   <xacro:macro name="beckhoff_bot" params="prefix parent *origin">
     <!-- LINKS -->
@@ -14,5 +14,5 @@
         <geometry>
           <cylinder length="0.3" radius="0.3"/>
-          <!--           <mesh filename="package://beckhoff_description/meshes/beckhoff_bot/visual/base_link.dae" /> -->
+          <!--           <mesh filename="package://beckhoff_bringup/meshes/beckhoff_bot/visual/base_link.dae" /> -->
         </geometry>
         <material name="black"/>
@@ -22,5 +22,5 @@
         <geometry>
           <cylinder length="0.3" radius="0.3"/>
-          <!--           <mesh filename="package://beckhoff_description/meshes/beckhoff_bot/collision/base_link.stl" /> -->
+          <!--           <mesh filename="package://beckhoff_bringup/meshes/beckhoff_bot/collision/base_link.stl" /> -->
         </geometry>
       </collision>
@@ -35,5 +35,5 @@
         <geometry>
           <cylinder length="0.3" radius="0.15"/>
-          <!--           <mesh filename="package://beckhoff_description/meshes/beckhoff_bot/visual/link1.dae" /> -->
+          <!--           <mesh filename="package://beckhoff_bringup/meshes/beckhoff_bot/visual/link1.dae" /> -->
         </geometry>
         <material name="blue"/>
@@ -43,5 +43,5 @@
         <geometry>
           <cylinder length="0.3" radius="0.15"/>
-          <!--           <mesh filename="package://beckhoff_description/meshes/beckhoff_bot/collision/link1.stl" /> -->
+          <!--           <mesh filename="package://beckhoff_bringup/meshes/beckhoff_bot/collision/link1.stl" /> -->
         </geometry>
         <material name="green"/>
@@ -57,5 +57,5 @@
         <geometry>
           <cylinder length="0.3" radius="0.15"/>
-          <!--           <mesh filename="package://beckhoff_description/meshes/beckhoff_bot/visual/link2.dae" /> -->
+          <!--           <mesh filename="package://beckhoff_bringup/meshes/beckhoff_bot/visual/link2.dae" /> -->
         </geometry>
         <material name="grey"/>
@@ -65,5 +65,5 @@
         <geometry>
           <cylinder length="0.3" radius="0.15"/>
-          <!--           <mesh filename="package://beckhoff_description/meshes/beckhoff_bot/collision/link2.stl"  /> -->
+          <!--           <mesh filename="package://beckhoff_bringup/meshes/beckhoff_bot/collision/link2.stl"  /> -->
         </geometry>
       </collision>
@@ -78,5 +78,5 @@
         <geometry>
           <cylinder length="0.2" radius="0.1"/>
-          <!--           <mesh filename="package://beckhoff_description/meshes/beckhoff_bot/visual/link3.dae" /> -->
+          <!--           <mesh filename="package://beckhoff_bringup/meshes/beckhoff_bot/visual/link3.dae" /> -->
         </geometry>
         <material name="orange"/>
@@ -86,5 +86,5 @@
         <geometry>
           <cylinder length="0.2" radius="0.1"/>
-          <!--           <mesh filename="package://beckhoff_description/meshes/beckhoff_bot/collision/link3.stl"  /> -->
+          <!--           <mesh filename="package://beckhoff_bringup/meshes/beckhoff_bot/collision/link3.stl"  /> -->
         </geometry>
       </collision>
@@ -99,5 +99,5 @@
         <geometry>
           <cylinder length="0.1" radius="0.1"/>
-          <!--           <mesh filename="package://beckhoff_description/meshes/beckhoff_bot/visual/link4.dae" /> -->
+          <!--           <mesh filename="package://beckhoff_bringup/meshes/beckhoff_bot/visual/link4.dae" /> -->
         </geometry>
         <material name="brown"/>
@@ -107,5 +107,5 @@
         <geometry>
           <cylinder length="0.1" radius="0.1"/>
-          <!--           <mesh filename="package://beckhoff_description/meshes/beckhoff_bot/collision/link4.stl"  /> -->
+          <!--           <mesh filename="package://beckhoff_bringup/meshes/beckhoff_bot/collision/link4.stl"  /> -->
         </geometry>
       </collision>
@@ -120,5 +120,5 @@
         <geometry>
           <cylinder length="0.15" radius="0.1"/>
-          <!--           <mesh filename="package://beckhoff_description/meshes/beckhoff_bot/visual/link5.dae" /> -->
+          <!--           <mesh filename="package://beckhoff_bringup/meshes/beckhoff_bot/visual/link5.dae" /> -->
         </geometry>
         <material name="red"/>
@@ -128,5 +128,5 @@
         <geometry>
           <cylinder length="0.15" radius="0.1"/>
-          <!--           <mesh filename="package://beckhoff_description/meshes/beckhoff_bot/collision/link5.stl" /> -->
+          <!--           <mesh filename="package://beckhoff_bringup/meshes/beckhoff_bot/collision/link5.stl" /> -->
         </geometry>
       </collision>
@@ -141,5 +141,5 @@
         <geometry>
           <cylinder length="0.05" radius="0.075"/>
-          <!--           <mesh filename="package://beckhoff_description/meshes/beckhoff_bot/visual/link6.dae" /> -->
+          <!--           <mesh filename="package://beckhoff_bringup/meshes/beckhoff_bot/visual/link6.dae" /> -->
         </geometry>
         <material name="white"/>
@@ -149,5 +149,5 @@
         <geometry>
           <cylinder length="0.05" radius="0.075"/>
-          <!--           <mesh filename="package://beckhoff_description/meshes/beckhoff_bot/collision/link6.stl" /> -->
+          <!--           <mesh filename="package://beckhoff_bringup/meshes/beckhoff_bot/collision/link6.stl" /> -->
         </geometry>
       </collision>
