Commit message: wrap beckhoff interfaces in a separate xacrp file

File: beckhoff_ads_bringup/urdf/beckhoff_bot/beckhoff_bot_macro.ros2_control.xacro (robot description, xacro)
@@ -1,27 +1,5 @@
 <?xml version="1.0" encoding="UTF-8"?>
 <robot xmlns:xacro="http://wiki.ros.org/xacro">
-    <xacro:macro name="command_interface_PLC" params="name initial_value:='' PLC_symbol PLC_type n_elements:=1 index:=''">
-        <command_interface name="${name}">
-            <xacro:if value="${initial_value != ''}">
-                <param name="initial_value">${initial_value}</param>
-            </xacro:if>
-            <param name="PLC_symbol">${PLC_symbol}</param>
-            <param name="PLC_type">${PLC_type}</param>
-            <param name="n_elements">${n_elements}</param>
-            <xacro:if value="${index != ''}">
-                <param name="index">${index}</param>
-            </xacro:if>
-        </command_interface>
-    </xacro:macro>
-    <xacro:macro name="state_interface_PLC" params="name PLC_symbol PLC_type n_elements:=1 index:=''">
-        <state_interface name="${name}">
-            <param name="PLC_symbol">${PLC_symbol}</param>
-            <param name="PLC_type">${PLC_type}</param>
-            <param name="n_elements">${n_elements}</param>
-            <xacro:if value="${index != ''}">
-                <param name="index">${index}</param>
-            </xacro:if>
-        </state_interface>
-    </xacro:macro>
+    <xacro:include filename="$(find beckhoff_bringup)/urdf/beckhoff_bot/beckhoff_ads_interfaces.ros2_control.xacro"/>
     <xacro:macro name="beckhoff_bot_ros2_control" params="
                 name
