Commit message: rename bringup package to beckhoff_ads_bringup

File: beckhoff_ads_bringup/urdf/beckhoff_bot.urdf.xacro (robot description, xacro)
@@ -4,6 +4,6 @@
   <xacro:arg name="mock_hardware" default="false"/>
   <xacro:arg name="mock_sensor_commands" default="false"/>
-  <xacro:include filename="$(find beckhoff_bringup)/urdf/beckhoff_bot/beckhoff_bot_macro.xacro"/>
-  <xacro:include filename="$(find beckhoff_bringup)/urdf/beckhoff_bot/beckhoff_bot_macro.ros2_control.xacro"/>
+  <xacro:include filename="$(find beckhoff_ads_bringup)/urdf/beckhoff_bot/beckhoff_bot_macro.xacro"/>
+  <xacro:include filename="$(find beckhoff_ads_bringup)/urdf/beckhoff_bot/beckhoff_bot_macro.ros2_control.xacro"/>
   <!-- create link fixed to the "world" -->
   <link name="world"/>

File: beckhoff_ads_bringup/urdf/beckhoff_bot/beckhoff_bot_macro.ros2_control.xacro (robot description, xacro)
@@ -1,5 +1,5 @@
 <?xml version="1.0" encoding="UTF-8"?>
 <robot xmlns:xacro="http://wiki.ros.org/xacro">
-    <xacro:include filename="$(find beckhoff_bringup)/urdf/beckhoff_bot/beckhoff_ads_interfaces.ros2_control.xacro"/>
+    <xacro:include filename="$(find beckhoff_ads_bringup)/urdf/beckhoff_bot/beckhoff_ads_interfaces.ros2_control.xacro"/>
     <xacro:macro name="beckhoff_bot_ros2_control" params="
                 name

File: beckhoff_ads_bringup/urdf/beckhoff_bot/beckhoff_bot_macro.xacro (robot description, xacro)
@@ -1,6 +1,6 @@
 <?xml version="1.0" encoding="UTF-8"?>
 <robot xmlns:xacro="http://wiki.ros.org/xacro">
-  <xacro:include filename="$(find beckhoff_bringup)/urdf/common/inertials.xacro"/>
-  <xacro:include filename="$(find beckhoff_bringup)/urdf/common/materials.xacro"/>
+  <xacro:include filename="$(find beckhoff_ads_bringup)/urdf/common/inertials.xacro"/>
+  <xacro:include filename="$(find beckhoff_ads_bringup)/urdf/common/materials.xacro"/>
   <xacro:macro name="beckhoff_bot" params="prefix parent *origin">
     <!-- LINKS -->
@@ -14,5 +14,5 @@
         <geometry>
           <cylinder length="0.3" radius="0.3"/>
-          <!--           <mesh filename="package://beckhoff_bringup/meshes/beckhoff_bot/visual/base_link.dae" /> -->
+          <!--           <mesh filename="package://beckhoff_ads_bringup/meshes/beckhoff_bot/visual/base_link.dae" /> -->
         </geometry>
         <material name="black"/>
@@ -22,5 +22,5 @@
         <geometry>
           <cylinder length="0.3" radius="0.3"/>
-          <!--           <mesh filename="package://beckhoff_bringup/meshes/beckhoff_bot/collision/base_link.stl" /> -->
+          <!--           <mesh filename="package://beckhoff_ads_bringup/meshes/beckhoff_bot/collision/base_link.stl" /> -->
         </geometry>
       </collision>
@@ -35,5 +35,5 @@
         <geometry>
           <cylinder length="0.3" radius="0.15"/>
-          <!--           <mesh filename="package://beckhoff_bringup/meshes/beckhoff_bot/visual/link1.dae" /> -->
+          <!--           <mesh filename="package://beckhoff_ads_bringup/meshes/beckhoff_bot/visual/link1.dae" /> -->
         </geometry>
         <material name="blue"/>
@@ -43,5 +43,5 @@
         <geometry>
           <cylinder length="0.3" radius="0.15"/>
-          <!--           <mesh filename="package://beckhoff_bringup/meshes/beckhoff_bot/collision/link1.stl" /> -->
+          <!--           <mesh filename="package://beckhoff_ads_bringup/meshes/beckhoff_bot/collision/link1.stl" /> -->
         </geometry>
         <material name="green"/>
@@ -57,5 +57,5 @@
         <geometry>
           <cylinder length="0.3" radius="0.15"/>
-          <!--           <mesh filename="package://beckhoff_bringup/meshes/beckhoff_bot/visual/link2.dae" /> -->
+          <!--           <mesh filename="package://beckhoff_ads_bringup/meshes/beckhoff_bot/visual/link2.dae" /> -->
         </geometry>
         <material name="grey"/>
@@ -65,5 +65,5 @@
         <geometry>
           <cylinder length="0.3" radius="0.15"/>
-          <!--           <mesh filename="package://beckhoff_bringup/meshes/beckhoff_bot/collision/link2.stl"  /> -->
+          <!--           <mesh filename="package://beckhoff_ads_bringup/meshes/beckhoff_bot/collision/link2.stl"  /> -->
         </geometry>
       </collision>
@@ -78,5 +78,5 @@
         <geometry>
           <cylinder length="0.2" radius="0.1"/>
-          <!--           <mesh filename="package://beckhoff_bringup/meshes/beckhoff_bot/visual/link3.dae" /> -->
+          <!--           <mesh filename="package://beckhoff_ads_bringup/meshes/beckhoff_bot/visual/link3.dae" /> -->
         </geometry>
         <material name="orange"/>
@@ -86,5 +86,5 @@
         <geometry>
           <cylinder length="0.2" radius="0.1"/>
-          <!--           <mesh filename="package://beckhoff_bringup/meshes/beckhoff_bot/collision/link3.stl"  /> -->
+          <!--           <mesh filename="package://beckhoff_ads_bringup/meshes/beckhoff_bot/collision/link3.stl"  /> -->
         </geometry>
       </collision>
@@ -99,5 +99,5 @@
         <geometry>
           <cylinder length="0.1" radius="0.1"/>
-          <!--           <mesh filename="package://beckhoff_bringup/meshes/beckhoff_bot/visual/link4.dae" /> -->
+          <!--           <mesh filename="package://beckhoff_ads_bringup/meshes/beckhoff_bot/visual/link4.dae" /> -->
         </geometry>
         <material name="brown"/>
@@ -107,5 +107,5 @@
         <geometry>
           <cylinder length="0.1" radius="0.1"/>
-          <!--           <mesh filename="package://beckhoff_bringup/meshes/beckhoff_bot/collision/link4.stl"  /> -->
+          <!--           <mesh filename="package://beckhoff_ads_bringup/meshes/beckhoff_bot/collision/link4.stl"  /> -->
         </geometry>
       </collision>
@@ -120,5 +120,5 @@
         <geometry>
           <cylinder length="0.15" radius="0.1"/>
-          <!--           <mesh filename="package://beckhoff_bringup/meshes/beckhoff_bot/visual/link5.dae" /> -->
+          <!--           <mesh filename="package://beckhoff_ads_bringup/meshes/beckhoff_bot/visual/link5.dae" /> -->
         </geometry>
         <material name="red"/>
@@ -128,5 +128,5 @@
         <geometry>
           <cylinder length="0.15" radius="0.1"/>
-          <!--           <mesh filename="package://beckhoff_bringup/meshes/beckhoff_bot/collision/link5.stl" /> -->
+          <!--           <mesh filename="package://beckhoff_ads_bringup/meshes/beckhoff_bot/collision/link5.stl" /> -->
         </geometry>
       </collision>
@@ -141,5 +141,5 @@
         <geometry>
           <cylinder length="0.05" radius="0.075"/>
-          <!--           <mesh filename="package://beckhoff_bringup/meshes/beckhoff_bot/visual/link6.dae" /> -->
+          <!--           <mesh filename="package://beckhoff_ads_bringup/meshes/beckhoff_bot/visual/link6.dae" /> -->
         </geometry>
         <material name="white"/>
@@ -149,5 +149,5 @@
         <geometry>
           <cylinder length="0.05" radius="0.075"/>
-          <!--           <mesh filename="package://beckhoff_bringup/meshes/beckhoff_bot/collision/link6.stl" /> -->
+          <!--           <mesh filename="package://beckhoff_ads_bringup/meshes/beckhoff_bot/collision/link6.stl" /> -->
         </geometry>
       </collision>
